File: Gateway/CSN-Gateway.sch (KiCad schematic (older format))
At the start: 63 parts, among them IC1 ATMEGA328-A, IC2 FT232RL, P1 USB_MINI, P2 CONN4, P3 CONN_ICSP, P4 CONN_OLED_SCREEN, P5 CONN6, P8 CONN_NRF24L01, Q1 2N2222, SW1 SW_PUSH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

Commit message: add 4th ct sensor input
Parts:
- added C20: 10uF, Capacitors_SMD:C_0805_HandSoldering, symbol C
- added R28: 33, Resistors_SMD:R_0805_HandSoldering, symbol R
- added R29, R30: 10K, Resistors_SMD:R_0805_HandSoldering, symbol R
- P2: symbol CONN4 -> CONN6
Connections:
- net GND: now also C20.2, R30.2
- net VCC: now also R29.2
- net A3: now reaches IC1.22 (ADC7)
- net A3: now also P2.5, R28.1
- new net CT1-A0: C20.1, P2.6, R28.2, R29.1, R30.1
- no-connect marks 15 -> 14
