File: Gateway/CSN-Gateway-base.kicad_pcb (KiCad board)
At the start: 2 copper layers, 32 x 85.5 mm, 56 parts, among them IC1 ATMEGA328-A, P1 CONN_02X06, P2 CONN4, P3 CONN_ICSP, P5 CONN6, Q1 2N2222, U1 MAX485CSA, U2 AMS1117-3.3V, U3 ATSHA204A, Y1 Crystal

Commit message: pin 4 of ams1117 to gnd
Connections:
- U2 pad 4: (no net) -> GND
Changed lines of the file:
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@@
 (kicad_pcb (version 4) (host pcbnew 4.0.4-stable)
   (general
-    (links 134)
+    (links 135)
     (no_connects 0)
     (area 109.424999 50.208999 141.575001 135.859008)
@@
       (padsonsilk false)
       (subtractmaskfromsilk false)
-      (outputformat 1)
+      (outputformat 4)
       (mirror false)
-      (drillshape 1)
+      (drillshape 2)
       (scaleselection 1)
       (outputdirectory ""))
@@
     (fp_line (start 2.032 -4.572) (end 3.556 -2.286) (layer F.SilkS) (width 0.15))
     (fp_line (start 3.556 -2.286) (end 3.556 -1.524) (layer F.SilkS) (width 0.15))
-    (pad 4 smd rect (at 0 -3.302) (size 3.6576 2.032) (layers F.Cu F.Paste F.Mask))
+    (pad 4 smd rect (at 0 -3.302) (size 3.6576 2.032) (layers F.Cu F.Paste F.Mask)
+      (net 2 GND))
     (pad 2 smd rect (at 0 3.302) (size 1.016 2.032) (layers F.Cu F.Paste F.Mask)
       (net 10 "Net-(C11-Pad1)"))
